File: 8x8x8LEDCube/8x8x8LEDCube.kicad_pcb (KiCad board)
At the start: 2 copper layers, 41 parts, among them P101 CONN_2, Q201 NPN, Q202 NPN, Q203 NPN, Q204 NPN, Q205 NPN, Q206 NPN, Q207 NPN, Q208 NPN, U201 SN74HC595DWR, U202 SN74HC595DWR, U203 SN74HC595DWR, U204 SN74HC595DWR, U205 SN74HC595DWR, U206 SN74HC595DWR, U207 SN74HC595DWR, U208 SN74HC595DWR

Commit message: Final version of the PCB
Parts:
- added C101: CONNECTOR_1X64, 1x64_Connector_Receptade_2.54mm, F.Cu at (246.5, 84.5)
- added C201: 0.1u, SM0805_NoVal, F.Cu at (170.8, 109.5)
- added C202: 0.1u, SM0805_NoVal, F.Cu at (193.3, 109.5)
- added C203: 0.1u, SM0805_NoVal, F.Cu at (213.5, 109.6)
- added C204: 0.1u, SM0805_NoVal, F.Cu at (234.1, 109.3)
- added C205: 0.1u, SM0805_NoVal, F.Cu at (254.9, 108.9)
- added C206: 0.1u, SM0805_NoVal, F.Cu at (274.9, 108.9)
- added C207: 0.1u, SM0805_NoVal, F.Cu at (295.2, 108.8)
- added C208: 0.1u, SM0805_NoVal, F.Cu at (315.5, 108.8)
- added C209: 47U, SM1210, B.Cu at (293.5, 127.0)
- added C210: 47U, SM1210, B.Cu at (242.6, 127.1)
- added C211: 0.1u, SM0805_NoVal, F.Cu at (177.2, 129.1)
- added C212: 47U, SM1210, B.Cu at (280.7, 127.1)
- added C213: 47U, SM1210, B.Cu at (229.8, 127.1)
- added C214: 47U, SM1210, B.Cu at (268.1, 127.1)
- added C215: 47U, SM1210, B.Cu at (217.0, 127.1)
- added C216: 47U, SM1210, B.Cu at (255.2, 127.1)
- added C217: 47U, SM1210, B.Cu at (204.4, 127.1)
- added K101: CONN_3, PIN_ARRAY_3X1, F.Cu at (160.1, 119.9)
- added P102: CONN_2, Terminal_Block_200mil_5mm, F.Cu at (324.2, 125.6)
- added P103: CONN_8, PIN_ARRAY_8x1, F.Cu at (308.2, 130.4)
- added Q209: NPN, SOT23_NPN_MMBT3904, B.Cu at (185.5, 88.9)
- added Q210: NPN, SOT23_NPN_MMBT3904, B.Cu at (188.0, 96.2)
- added Q211: NPN, SOT23_NPN_MMBT3904, B.Cu at (190.6, 88.9)
- added Q212: NPN, SOT23_NPN_MMBT3904, B.Cu at (193.1, 96.2)
- added Q213: NPN, SOT23_NPN_MMBT3904, B.Cu at (195.7, 89.0)
- added Q214: NPN, SOT23_NPN_MMBT3904, B.Cu at (198.2, 96.2)
- added Q215: NPN, SOT23_NPN_MMBT3904, B.Cu at (200.8, 89.0)
- added Q216: NPN, SOT23_NPN_MMBT3904, B.Cu at (203.3, 96.2)
- added Q217: NPN, SOT23_NPN_MMBT3904, B.Cu at (205.9, 89.0)
- added Q218: NPN, SOT23_NPN_MMBT3904, B.Cu at (208.3, 96.1)
- added Q219: NPN, SOT23_NPN_MMBT3904, B.Cu at (210.9, 89.0)
- added Q220: NPN, SOT23_NPN_MMBT3904, B.Cu at (213.4, 96.1)
- added Q221: NPN, SOT23_NPN_MMBT3904, B.Cu at (216.0, 89.0)
- added Q222: NPN, SOT23_NPN_MMBT3904, B.Cu at (218.5, 96.1)
- added Q223: NPN, SOT23_NPN_MMBT3904, B.Cu at (221.1, 89.0)
- added Q224: NPN, SOT23_NPN_MMBT3904, B.Cu at (223.6, 96.2)
- added Q225: NPN, SOT23_NPN_MMBT3904, B.Cu at (226.1, 89.0)
- added Q226: NPN, SOT23_NPN_MMBT3904, B.Cu at (228.7, 96.1)
- added Q227: NPN, SOT23_NPN_MMBT3904, B.Cu at (231.2, 88.9)
- added Q228: NPN, SOT23_NPN_MMBT3904, B.Cu at (233.8, 96.1)
- added Q229: NPN, SOT23_NPN_MMBT3904, B.Cu at (236.3, 88.9)
- added Q230: NPN, SOT23_NPN_MMBT3904, B.Cu at (238.8, 96.1)
- added Q231: NPN, SOT23_NPN_MMBT3904, B.Cu at (241.4, 88.9)
- added Q232: NPN, SOT23_NPN_MMBT3904, B.Cu at (243.9, 96.2)
- added Q233: NPN, SOT23_NPN_MMBT3904, B.Cu at (246.5, 88.9)
- added Q234: NPN, SOT23_NPN_MMBT3904, B.Cu at (249.0, 96.1)
- added Q235: NPN, SOT23_NPN_MMBT3904, B.Cu at (251.6, 88.9)
- added Q236: NPN, SOT23_NPN_MMBT3904, B.Cu at (254.1, 96.1)
- added Q237: NPN, SOT23_NPN_MMBT3904, B.Cu at (256.6, 88.9)
- added Q238: NPN, SOT23_NPN_MMBT3904, B.Cu at (259.2, 96.1)
- added Q239: NPN, SOT23_NPN_MMBT3904, B.Cu at (261.7, 88.9)
- added Q240: NPN, SOT23_NPN_MMBT3904, B.Cu at (264.3, 96.1)
- added Q241: NPN, SOT23_NPN_MMBT3904, B.Cu at (266.8, 88.9)
- added Q242: NPN, SOT23_NPN_MMBT3904, B.Cu at (269.3, 96.1)
- added Q243: NPN, SOT23_NPN_MMBT3904, B.Cu at (271.9, 88.9)
- added Q244: NPN, SOT23_NPN_MMBT3904, B.Cu at (274.4, 96.1)
- added Q245: NPN, SOT23_NPN_MMBT3904, B.Cu at (277.0, 88.9)
- added Q246: NPN, SOT23_NPN_MMBT3904, B.Cu at (279.5, 96.1)
- added Q247: NPN, SOT23_NPN_MMBT3904, B.Cu at (282.0, 88.9)
- added Q248: NPN, SOT23_NPN_MMBT3904, B.Cu at (284.6, 96.1)
- added Q249: NPN, SOT23_NPN_MMBT3904, B.Cu at (287.1, 88.9)
- added Q250: NPN, SOT23_NPN_MMBT3904, B.Cu at (289.7, 96.1)
- added Q251: NPN, SOT23_NPN_MMBT3904, B.Cu at (292.2, 88.9)
- added Q252: NPN, SOT23_NPN_MMBT3904, B.Cu at (294.8, 96.1)
- added Q253: NPN, SOT23_NPN_MMBT3904, B.Cu at (297.3, 88.9)
- added Q254: NPN, SOT23_NPN_MMBT3904, B.Cu at (299.8, 96.1)
- added Q255: NPN, SOT23_NPN_MMBT3904, B.Cu at (302.3, 88.9)
- added Q256: NPN, SOT23_NPN_MMBT3904, B.Cu at (304.9, 96.1)
- added Q257: NPN, SOT23_NPN_MMBT3904, B.Cu at (307.4, 88.9)
- added Q258: NPN, SOT23_NPN_MMBT3904, B.Cu at (310.0, 96.1)
- added Q259: NPN, SOT23_NPN_MMBT3904, B.Cu at (312.5, 88.9)
- added Q260: NPN, SOT23_NPN_MMBT3904, B.Cu at (315.1, 96.1)
- added Q261: NPN, SOT23_NPN_MMBT3904, B.Cu at (317.6, 88.9)
- added Q262: NPN, SOT23_NPN_MMBT3904, B.Cu at (320.1, 96.1)
- added Q263: NPN, SOT23_NPN_MMBT3904, B.Cu at (322.7, 88.9)
- added Q264: NPN, SOT23_NPN_MMBT3904, B.Cu at (325.2, 96.1)
- added Q265: NPN, SOT23_NPN_MMBT3904, B.Cu at (287.3, 127.3)
- added Q266: NPN, SOT23_NPN_MMBT3904, B.Cu at (236.7, 127.3)
- added Q267: IRF9540N, TO220_IRF9540N, F.Cu at (290.8, 132.3)
- added Q268: IRF9540N, TO220_IRF9540N, F.Cu at (239.8, 132.3)
- added Q269: NPN, SOT23_NPN_MMBT3904, B.Cu at (274.5, 127.4)
- added Q270: NPN, SOT23_NPN_MMBT3904, B.Cu at (223.8, 127.3)
- added Q271: IRF9540N, TO220_IRF9540N, F.Cu at (278.1, 132.4)
- added Q272: IRF9540N, TO220_IRF9540N, F.Cu at (227.0, 132.3)
- added Q273: NPN, SOT23_NPN_MMBT3904, B.Cu at (261.9, 127.3)
- added Q274: NPN, SOT23_NPN_MMBT3904, B.Cu at (210.7, 127.3)
- added Q275: IRF9540N, TO220_IRF9540N, F.Cu at (265.3, 132.3)
- added Q276: IRF9540N, TO220_IRF9540N, F.Cu at (214.2, 132.3)
- added Q277: NPN, SOT23_NPN_MMBT3904, B.Cu at (249.3, 127.3)
- added Q278: NPN, SOT23_NPN_MMBT3904, B.Cu at (198.1, 127.3)
- added Q279: IRF9540N, TO220_IRF9540N, F.Cu at (252.5, 132.3)
- added Q280: IRF9540N, TO220_IRF9540N, F.Cu at (201.5, 132.3)
- added R101: 0, SM0805_NoVal, B.Cu at (321.2, 117.3)
- added R225: 100, SM0805_NoVal, F.Cu at (170.3, 88.3)
- added R226: 1K, SM0805_NoVal, F.Cu at (173.8, 98.9)
- added R227: 1K, SM0805_NoVal, F.Cu at (171.7, 98.9)
- added R228: 100, SM0805_NoVal, F.Cu at (172.8, 95.4)
- added R229: 1K, SM0805_NoVal, F.Cu at (176.3, 91.7)
- added R230: 1K, SM0805_NoVal, F.Cu at (174.2, 91.7)
- added R231: 100, SM0805_NoVal, F.Cu at (175.4, 88.2)
- added R232: 1K, SM0805_NoVal, F.Cu at (178.9, 98.9)
- added R233: 1K, SM0805_NoVal, F.Cu at (176.9, 98.9)
- added R234: 100, SM0805_NoVal, F.Cu at (177.9, 95.5)
- added R235: 1K, SM0805_NoVal, F.Cu at (181.4, 91.7)
- added R236: 1K, SM0805_NoVal, F.Cu at (179.4, 91.7)
- added R237: 100, SM0805_NoVal, F.Cu at (180.5, 88.4)
- added R238: 1K, SM0805_NoVal, F.Cu at (183.9, 98.9)
- added R239: 1K, SM0805_NoVal, F.Cu at (181.9, 98.9)
- added R240: 100, SM0805_NoVal, F.Cu at (183.0, 95.5)
- added R241: 1K, SM0805_NoVal, F.Cu at (186.5, 91.7)
- added R242: 1K, SM0805_NoVal, F.Cu at (184.6, 91.7)
- added R243: 100, SM0805_NoVal, F.Cu at (185.5, 88.2)
- added R244: 1K, SM0805_NoVal, F.Cu at (189.1, 98.9)
- added R245: 1K, SM0805_NoVal, F.Cu at (187.1, 98.9)
- added R246: 100, SM0805_NoVal, F.Cu at (188.1, 95.5)
- added R247: 1K, SM0805_NoVal, F.Cu at (191.6, 91.7)
- added R248: 1K, SM0805_NoVal, F.Cu at (189.6, 91.7)
- added R249: 100, SM0805_NoVal, F.Cu at (190.6, 88.2)
- added R250: 1K, SM0805_NoVal, F.Cu at (194.1, 98.9)
- added R251: 1K, SM0805_NoVal, F.Cu at (192.1, 98.9)
- added R252: 100, SM0805_NoVal, F.Cu at (193.1, 95.5)
- added R253: 1K, SM0805_NoVal, F.Cu at (196.7, 91.7)
- added R254: 1K, SM0805_NoVal, F.Cu at (194.7, 91.7)
- added R255: 100, SM0805_NoVal, F.Cu at (195.7, 88.2)
- added R256: 1K, SM0805_NoVal, F.Cu at (199.2, 98.9)
- added R257: 1K, SM0805_NoVal, F.Cu at (197.2, 98.9)
- added R258: 100, SM0805_NoVal, F.Cu at (198.2, 95.5)
- added R259: 1K, SM0805_NoVal, F.Cu at (201.8, 91.7)
- added R260: 1K, SM0805_NoVal, F.Cu at (199.7, 91.7)
- added R261: 100, SM0805_NoVal, F.Cu at (200.8, 88.2)
- added R262: 1K, SM0805_NoVal, F.Cu at (204.2, 98.9)
- added R263: 1K, SM0805_NoVal, F.Cu at (202.3, 98.9)
- added R264: 100, SM0805_NoVal, F.Cu at (203.3, 95.5)
- added R265: 1K, SM0805_NoVal, F.Cu at (206.8, 91.7)
- added R266: 1K, SM0805_NoVal, F.Cu at (204.7, 91.7)
- added R267: 100, SM0805_NoVal, F.Cu at (205.9, 88.2)
- added R268: 1K, SM0805_NoVal, F.Cu at (209.4, 98.9)
- added R269: 1K, SM0805_NoVal, F.Cu at (207.4, 98.9)
- added R270: 100, SM0805_NoVal, F.Cu at (208.4, 95.5)
- added R271: 1K, SM0805_NoVal, F.Cu at (211.9, 91.7)
- added R272: 1K, SM0805_NoVal, F.Cu at (209.9, 91.7)
- added R273: 100, SM0805_NoVal, F.Cu at (210.9, 88.2)
- added R274: 1K, SM0805_NoVal, F.Cu at (214.3, 98.9)
- added R275: 1K, SM0805_NoVal, F.Cu at (212.4, 98.9)
- added R276: 100, SM0805_NoVal, F.Cu at (213.5, 95.5)
- added R277: 1K, SM0805_NoVal, F.Cu at (217.0, 91.7)
- added R278: 1K, SM0805_NoVal, F.Cu at (215.0, 91.7)
- added R279: 100, SM0805_NoVal, F.Cu at (216.0, 88.2)
- added R280: 1K, SM0805_NoVal, F.Cu at (219.5, 98.9)
- added R281: 1K, SM0805_NoVal, F.Cu at (217.5, 98.9)
- added R282: 100, SM0805_NoVal, F.Cu at (218.5, 95.5)
- added R283: 1K, SM0805_NoVal, F.Cu at (222.0, 91.7)
- added R284: 1K, SM0805_NoVal, F.Cu at (220.1, 91.7)
- added R285: 100, SM0805_NoVal, F.Cu at (221.1, 88.2)
- added R286: 1K, SM0805_NoVal, F.Cu at (224.6, 98.9)
- added R287: 1K, SM0805_NoVal, F.Cu at (222.7, 98.9)
- added R288: 100, SM0805_NoVal, F.Cu at (223.6, 95.5)
- added R289: 1K, SM0805_NoVal, F.Cu at (227.0, 91.7)
- added R290: 1K, SM0805_NoVal, F.Cu at (225.2, 91.7)
- added R291: 100, SM0805_NoVal, F.Cu at (226.2, 88.2)
- added R292: 1K, SM0805_NoVal, F.Cu at (229.5, 98.9)
- added R293: 1K, SM0805_NoVal, F.Cu at (227.6, 98.9)
- added R294: 100, SM0805_NoVal, F.Cu at (228.7, 95.5)
- added R295: 1K, SM0805_NoVal, F.Cu at (232.1, 91.7)
- added R296: 1K, SM0805_NoVal, F.Cu at (230.2, 91.7)
- added R297: 100, SM0805_NoVal, F.Cu at (231.2, 88.2)
- added R298: 1K, SM0805_NoVal, F.Cu at (234.8, 98.9)
- added R299: 1K, SM0805_NoVal, F.Cu at (232.9, 98.9)
- added R300: 100, SM0805_NoVal, F.Cu at (233.8, 95.5)
- added R301: 1K, SM0805_NoVal, F.Cu at (237.2, 91.7)
- added R302: 1K, SM0805_NoVal, F.Cu at (235.2, 91.7)
- added R303: 100, SM0805_NoVal, F.Cu at (236.3, 88.2)
- added R304: 1K, SM0805_NoVal, F.Cu at (239.9, 98.9)
- added R305: 1K, SM0805_NoVal, F.Cu at (237.9, 98.9)
- added R306: 100, SM0805_NoVal, F.Cu at (238.9, 95.5)
- added R307: 1K, SM0805_NoVal, F.Cu at (242.3, 91.7)
- added R308: 1K, SM0805_NoVal, F.Cu at (240.3, 91.7)
- added R309: 100, SM0805_NoVal, F.Cu at (241.4, 88.2)
- added R310: 1K, SM0805_NoVal, F.Cu at (244.9, 98.9)
- added R311: 1K, SM0805_NoVal, F.Cu at (243.0, 98.9)
- added R312: 100, SM0805_NoVal, F.Cu at (243.9, 95.5)
- added R313: 1K, SM0805_NoVal, F.Cu at (247.5, 91.7)
- added R314: 1K, SM0805_NoVal, F.Cu at (245.5, 91.7)
- added R315: 100, SM0805_NoVal, F.Cu at (246.5, 88.2)
- added R316: 1K, SM0805_NoVal, F.Cu at (250.0, 98.9)
- added R317: 1K, SM0805_NoVal, F.Cu at (248.0, 98.9)
- added R318: 100, SM0805_NoVal, F.Cu at (249.0, 95.5)
- added R319: 1K, SM0805_NoVal, F.Cu at (252.6, 91.7)
- added R320: 1K, SM0805_NoVal, F.Cu at (250.7, 91.7)
- added R321: 100, SM0805_NoVal, F.Cu at (251.6, 88.2)
- added R322: 1K, SM0805_NoVal, F.Cu at (255.0, 98.9)
- added R323: 1K, SM0805_NoVal, F.Cu at (253.1, 98.9)
- added R324: 100, SM0805_NoVal, F.Cu at (254.1, 95.5)
- added R325: 1K, SM0805_NoVal, F.Cu at (257.5, 91.7)
- added R326: 1K, SM0805_NoVal, F.Cu at (255.6, 91.7)
- added R327: 100, SM0805_NoVal, F.Cu at (256.6, 88.2)
- added R328: 1K, SM0805_NoVal, F.Cu at (260.1, 98.9)
- added R329: 1K, SM0805_NoVal, F.Cu at (258.1, 98.9)
- added R330: 100, SM0805_NoVal, F.Cu at (259.2, 95.5)
- added R331: 1K, SM0805_NoVal, F.Cu at (262.7, 91.7)
- added R332: 1K, SM0805_NoVal, F.Cu at (260.8, 91.7)
- added R333: 100, SM0805_NoVal, F.Cu at (261.7, 88.2)
- added R334: 1K, SM0805_NoVal, F.Cu at (265.2, 98.9)
- added R335: 1K, SM0805_NoVal, F.Cu at (263.2, 98.9)
- added R336: 100, SM0805_NoVal, F.Cu at (264.3, 95.5)
- added R337: 1K, SM0805_NoVal, F.Cu at (267.8, 91.7)
- added R338: 1K, SM0805_NoVal, F.Cu at (265.8, 91.7)
- added R339: 100, SM0805_NoVal, F.Cu at (266.8, 88.2)
- added R340: 1K, SM0805_NoVal, F.Cu at (270.3, 98.9)
- added R341: 1K, SM0805_NoVal, F.Cu at (268.4, 98.9)
- added R342: 100, SM0805_NoVal, F.Cu at (269.3, 95.5)
- added R343: 1K, SM0805_NoVal, F.Cu at (272.8, 91.7)
- added R344: 1K, SM0805_NoVal, F.Cu at (270.8, 91.7)
- added R345: 100, SM0805_NoVal, F.Cu at (271.9, 88.2)
- added R346: 1K, SM0805_NoVal, F.Cu at (275.3, 98.9)
- added R347: 1K, SM0805_NoVal, F.Cu at (273.3, 98.9)
- added R348: 100, SM0805_NoVal, F.Cu at (274.4, 95.5)
- added R349: 1K, SM0805_NoVal, F.Cu at (277.9, 91.7)
- added R350: 1K, SM0805_NoVal, F.Cu at (276.0, 91.7)
- added R351: 100, SM0805_NoVal, F.Cu at (277.0, 88.2)
- added R352: 1K, SM0805_NoVal, F.Cu at (280.5, 98.9)
- added R353: 1K, SM0805_NoVal, F.Cu at (278.6, 98.9)
- added R354: 100, SM0805_NoVal, F.Cu at (279.5, 95.5)
- added R355: 1K, SM0805_NoVal, F.Cu at (283.0, 91.7)
- added R356: 1K, SM0805_NoVal, F.Cu at (281.1, 91.7)
- added R357: 100, SM0805_NoVal, F.Cu at (282.0, 88.2)
- added R358: 1K, SM0805_NoVal, F.Cu at (285.5, 98.9)
- added R359: 1K, SM0805_NoVal, F.Cu at (283.5, 98.9)
- added R360: 100, SM0805_NoVal, F.Cu at (284.6, 95.5)
- added R361: 1K, SM0805_NoVal, F.Cu at (288.1, 91.7)
- added R362: 1K, SM0805_NoVal, F.Cu at (286.2, 91.7)
- added R363: 100, SM0805_NoVal, F.Cu at (287.1, 88.2)
- added R364: 1K, SM0805_NoVal, F.Cu at (290.7, 98.9)
- added R365: 1K, SM0805_NoVal, F.Cu at (288.7, 98.9)
- added R366: 100, SM0805_NoVal, F.Cu at (289.7, 95.5)
- added R367: 1K, SM0805_NoVal, F.Cu at (293.1, 91.7)
- added R368: 1K, SM0805_NoVal, F.Cu at (291.1, 91.7)
- added R369: 100, SM0805_NoVal, F.Cu at (292.2, 88.2)
- added R370: 1K, SM0805_NoVal, F.Cu at (295.8, 98.9)
- added R371: 1K, SM0805_NoVal, F.Cu at (293.8, 98.9)
- added R372: 100, SM0805_NoVal, F.Cu at (294.8, 95.5)
- added R373: 1K, SM0805_NoVal, F.Cu at (298.2, 91.7)
- added R374: 1K, SM0805_NoVal, F.Cu at (296.2, 91.7)
- added R375: 100, SM0805_NoVal, F.Cu at (297.3, 88.2)
- added R376: 1K, SM0805_NoVal, F.Cu at (300.8, 98.9)
- added R377: 1K, SM0805_NoVal, F.Cu at (298.8, 98.9)
- added R378: 100, SM0805_NoVal, F.Cu at (299.8, 95.5)
- added R379: 1K, SM0805_NoVal, F.Cu at (303.5, 91.7)
- added R380: 1K, SM0805_NoVal, F.Cu at (301.5, 91.7)
- added R381: 100, SM0805_NoVal, F.Cu at (302.4, 88.2)
- added R382: 1K, SM0805_NoVal, F.Cu at (305.9, 98.9)
- added R383: 1K, SM0805_NoVal, F.Cu at (304.0, 98.9)
- added R384: 100, SM0805_NoVal, F.Cu at (304.9, 95.5)
- added R385: 1K, SM0805_NoVal, F.Cu at (308.3, 91.7)
- added R386: 1K, SM0805_NoVal, F.Cu at (306.4, 91.7)
- added R387: 100, SM0805_NoVal, F.Cu at (307.4, 88.2)
- added R388: 1K, SM0805_NoVal, F.Cu at (310.8, 98.9)
- added R389: 1K, SM0805_NoVal, F.Cu at (308.9, 98.9)
- added R390: 100, SM0805_NoVal, F.Cu at (310.0, 95.5)
- added R391: 1K, SM0805_NoVal, F.Cu at (313.5, 91.7)
- added R392: 1K, SM0805_NoVal, F.Cu at (311.6, 91.7)
- added R393: 100, SM0805_NoVal, F.Cu at (312.5, 88.2)
- added R394: 1K, SM0805_NoVal, F.Cu at (316.0, 98.9)
- added R395: 1K, SM0805_NoVal, F.Cu at (314.1, 98.9)
- added R396: 100, SM0805_NoVal, F.Cu at (315.1, 95.5)
- added R397: 1K, SM0805_NoVal, F.Cu at (318.6, 91.7)
- added R398: 1K, SM0805_NoVal, F.Cu at (316.7, 91.7)
- added R399: 100, SM0805_NoVal, F.Cu at (317.6, 88.2)
- added R400: 1K, SM0805_NoVal, F.Cu at (321.2, 98.9)
- added R401: 1K, SM0805_NoVal, F.Cu at (319.3, 98.9)
- added R402: 100, SM0805_NoVal, F.Cu at (320.2, 95.5)
- added R403: 1K, SM0805_NoVal, F.Cu at (323.7, 91.7)
- added R404: 1K, SM0805_NoVal, F.Cu at (321.7, 91.7)
- added R405: 100, SM0805_NoVal, F.Cu at (322.7, 88.2)
- added R406: 1K, SM0805_NoVal, F.Cu at (326.2, 98.9)
- added R407: 1K, SM0805_NoVal, F.Cu at (324.3, 98.9)
- added R408: 100, SM0805_NoVal, F.Cu at (325.2, 95.5)
- added R409: 0, SM0805_NoVal, B.Cu at (266.9, 117.1)
- added R410: 0, SM0805_NoVal, B.Cu at (286.5, 117.1)
- added R411: 0, SM0805_NoVal, B.Cu at (307.0, 117.1)
- added R412: 0, SM0805_NoVal, B.Cu at (205.6, 117.1)
- added R413: 0, SM0805_NoVal, B.Cu at (226.0, 117.1)
- added R414: 0, SM0805_NoVal, B.Cu at (246.6, 117.1)
- added R415: 0, SM0805_NoVal, B.Cu at (184.5, 117.1)
- added R416: 0, SM0805_NoVal, F.Cu at (167.1, 117.3)
- added R417: 1K, SM0805_NoVal, F.Cu at (287.6, 126.4)
- added R418: 1K, SM0805_NoVal, F.Cu at (236.8, 126.4)
- added R419: 1K, SM0805_NoVal, F.Cu at (289.6, 126.4)
- added R420: 1K, SM0805_NoVal, F.Cu at (238.8, 126.4)
- added R421: 100, SM0805_NoVal, B.Cu at (290.9, 127.2)
- added R422: 100, SM0805_NoVal, B.Cu at (239.9, 127.2)
- added R423: 1K, SM0805_NoVal, F.Cu at (274.8, 126.4)
- added R424: 1K, SM0805_NoVal, F.Cu at (223.9, 126.4)
- added R425: 1K, SM0805_NoVal, F.Cu at (276.8, 126.4)
- added R426: 1K, SM0805_NoVal, F.Cu at (225.9, 126.4)
- added R427: 0, SM0805_NoVal, F.Cu at (166.1, 122.3)
- added R428: 0, SM0805_NoVal, F.Cu at (173.0, 130.1)
- added R429: 0, SM0805_NoVal, F.Cu at (177.2, 131.1)
- added R430: 100, SM0805_NoVal, B.Cu at (278.1, 127.2)
- added R431: 100, SM0805_NoVal, B.Cu at (227.0, 127.2)
- added R432: 1K, SM0805_NoVal, F.Cu at (262.1, 126.4)
- added R433: 1K, SM0805_NoVal, F.Cu at (210.9, 126.4)
- added R434: 1K, SM0805_NoVal, F.Cu at (264.1, 126.4)
- added R435: 1K, SM0805_NoVal, F.Cu at (212.9, 126.4)
- added R436: 100, SM0805_NoVal, B.Cu at (265.3, 127.2)
- added R437: 100, SM0805_NoVal, B.Cu at (214.2, 127.2)
- added R438: 1K, SM0805_NoVal, F.Cu at (249.3, 126.4)
- added R439: 1K, SM0805_NoVal, F.Cu at (198.3, 126.4)
- added R440: 1K, SM0805_NoVal, F.Cu at (251.3, 126.4)
- added R441: 1K, SM0805_NoVal, F.Cu at (200.3, 126.4)
- added R442: 100, SM0805_NoVal, B.Cu at (252.5, 127.2)
- added R443: 100, SM0805_NoVal, B.Cu at (201.5, 127.2)
- added R444: 0, SM0805_NoVal, F.Cu at (168.4, 122.3)
- added U209: SN74HC595DWR, SOIC16_SN74HC595DWR, B.Cu at (176.5, 130.0)
- Q201, Q202, Q203, Q204, Q205, Q206, Q207, Q208: footprint SOT23 -> SOT23_NPN_MMBT3904; moved to B.Cu
- R201, R202, R204, R205, R207, R208, R210, R211, R213, R214, R216: value 1K -> 0; footprint SM0805 -> SM0805_NoVal
- R203, R206, R209, R212, R215: value 100 -> 0; footprint SM0805 -> SM0805_NoVal
- R217, R220, R223: footprint SM0805 -> SM0805_NoVal
- R218, R221, R224: value 100 -> 1K; footprint SM0805 -> SM0805_NoVal
- R219, R222: value 1K -> 100; footprint SM0805 -> SM0805_NoVal
- U201, U202, U203, U204, U205, U206, U207, U208: moved to B.Cu
- moved R215 273.4 mm to (316.5, 113.2)
- moved U207 246.0 mm to (296.4, 109.8), turned to 270 degrees
- moved U208 224.6 mm to (316.5, 109.8), turned to 270 degrees
- moved R214 210.4 mm to (297.3, 108.8), turned to 270 degrees
- moved R213 206.7 mm to (296.5, 113.2)
- moved R212 201.1 mm to (276.9, 108.9), turned to 270 degrees
- moved R211 193.9 mm to (276.2, 113.2)
- moved R216 190.8 mm to (317.4, 108.8), turned to 270 degrees
- moved R209 188.6 mm to (256.2, 113.3)
- moved R210 178.0 mm to (257.1, 108.9), turned to 270 degrees
- moved R207 164.4 mm to (235.2, 113.4)
- moved R206 158.6 mm to (215.5, 109.6), turned to 270 degrees
- moved U203 156.7 mm to (214.6, 109.8), turned to 270 degrees
- moved U204 156.3 mm to (235.2, 109.8), turned to 270 degrees
- moved U205 156.2 mm to (256.0, 109.8), turned to 270 degrees
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Connections:
- Q201 pad 2: N-0000022 -> N-00000256
- Q201 pad 3: N-0000021 -> N-00000247
- Q202 pad 2: N-0000019 -> N-00000245
- Q202 pad 3: N-0000018 -> N-00000244
- Q203 pad 2: N-0000016 -> N-00000242
- Q203 pad 3: N-0000015 -> N-00000241
- Q204 pad 2: N-0000037 -> N-00000239
- Q204 pad 3: N-0000036 -> N-00000238
- Q205 pad 2: N-0000034 -> N-00000236
- Q205 pad 3: N-0000033 -> N-00000235
- Q206 pad 2: N-0000031 -> N-00000233
- Q206 pad 3: N-0000039 -> N-00000265
- Q207 pad 2: N-0000026 -> N-00000252
- Q207 pad 3: N-0000029 -> N-00000251
- Q208 pad 2: N-0000028 -> N-00000249
- Q208 pad 3: N-0000027 -> N-00000248
- R201 pad 1: RedC1 -> VCC
- R201 pad 2: N-0000022 -> N-00000264
- R202 pad 1: VCC -> GND
- R202 pad 2: N-0000021 -> N-00000263
- R203 pad 1: N-0000021 -> VCC
- R203 pad 2: (no net) -> N-00000272
- R204 pad 1: RedC2 -> GND
- R204 pad 2: N-0000019 -> N-00000266
- R205 pad 2: N-0000018 -> N-00000303
- R206 pad 1: N-0000018 -> GND
- R206 pad 2: (no net) -> N-00000268
- R207 pad 1: RedC3 -> VCC
- R207 pad 2: N-0000016 -> N-00000267
- R208 pad 1: VCC -> GND
- R208 pad 2: N-0000015 -> N-00000271
- R209 pad 1: N-0000015 -> VCC
- R209 pad 2: (no net) -> N-00000270
- R210 pad 1: RedC4 -> GND
- R210 pad 2: N-0000037 -> N-00000269
- R211 pad 2: N-0000036 -> N-00000301
- R212 pad 1: N-0000036 -> GND
- R212 pad 2: (no net) -> N-00000274
- R213 pad 1: RedC5 -> VCC
- R213 pad 2: N-0000034 -> N-00000273
- R214 pad 1: VCC -> GND
- R214 pad 2: N-0000033 -> N-00000302
- R215 pad 1: N-0000033 -> VCC
- R215 pad 2: (no net) -> N-00000276
- R216 pad 1: RedC6 -> GND
- R216 pad 2: N-0000031 -> N-00000275
- R217 pad 1: VCC -> RedC1
- R217 pad 2: N-0000039 -> N-00000256
- R218 pad 1: N-0000039 -> VCC
- R218 pad 2: (no net) -> N-00000247
- R219 pad 1: RedC7 -> N-00000247
- R219 pad 2: N-0000026 -> /ColorControl/C1Red
- R220 pad 1: VCC -> RedC2
- R220 pad 2: N-0000029 -> N-00000245
- R221 pad 1: N-0000029 -> VCC
- R221 pad 2: (no net) -> N-00000244
- R222 pad 1: RedC8 -> N-00000244
- R222 pad 2: N-0000028 -> /ColorControl/C2Red
- R223 pad 1: VCC -> RedC3
- R223 pad 2: N-0000027 -> N-00000242
- R224 pad 1: N-0000027 -> VCC
- R224 pad 2: (no net) -> N-00000241
- U201 pad 10: VCC -> N-00000264
- U201 pad 13: GND -> N-00000263
- U201 pad 14: (no net) -> N-00000201
- U201 pad 9: N-0000083 -> N-00000202
- U202 pad 1: (no net) -> RedC10
- U202 pad 10: VCC -> N-00000272
- U202 pad 13: GND -> N-00000266
- U202 pad 14: N-0000083 -> N-00000253
- U202 pad 15: (no net) -> RedC9
- U202 pad 2: (no net) -> RedC11
- U202 pad 3: (no net) -> RedC12
- U202 pad 4: (no net) -> RedC13
- U202 pad 5: (no net) -> RedC14
- U202 pad 6: (no net) -> RedC15
- U202 pad 7: (no net) -> RedC16
- U202 pad 9: N-0000058 -> N-00000254
- U203 pad 1: (no net) -> RedC18
- U203 pad 10: VCC -> N-00000303
- U203 pad 13: GND -> N-00000268
- U203 pad 14: N-0000058 -> N-00000262
- U203 pad 15: (no net) -> RedC17
- U203 pad 2: (no net) -> RedC19
- U203 pad 3: (no net) -> RedC20
- U203 pad 4: (no net) -> RedC21
- U203 pad 5: (no net) -> RedC22
- U203 pad 6: (no net) -> RedC23
- U203 pad 7: (no net) -> RedC24
- U203 pad 9: N-0000048 -> N-00000196
- U204 pad 1: (no net) -> RedC26
- U204 pad 10: VCC -> N-00000267
- U204 pad 13: (no net) -> N-00000271
- U204 pad 14: N-0000048 -> N-00000261
- U204 pad 15: (no net) -> RedC25
- U204 pad 2: (no net) -> RedC27
- U204 pad 3: (no net) -> RedC28
- U204 pad 4: (no net) -> RedC29
- U204 pad 5: (no net) -> RedC30
- U204 pad 6: (no net) -> RedC31
- U204 pad 7: (no net) -> RedC32
- U204 pad 9: N-0000092 -> N-00000197
- U205 pad 1: (no net) -> RedC34
- U205 pad 10: VCC -> N-00000270
- U205 pad 13: GND -> N-00000269
- U205 pad 14: N-0000092 -> N-00000260
- U205 pad 15: (no net) -> RedC33
- U205 pad 2: (no net) -> RedC35
- U205 pad 3: (no net) -> RedC36
- U205 pad 4: (no net) -> RedC37
- U205 pad 5: (no net) -> RedC38
- U205 pad 6: (no net) -> RedC39
- U205 pad 7: (no net) -> RedC40
- U205 pad 9: N-0000025 -> N-00000198
- U206 pad 1: (no net) -> RedC42
- U206 pad 10: VCC -> N-00000301
- U206 pad 13: GND -> N-00000274
- U206 pad 14: N-0000025 -> N-00000259
- U206 pad 15: (no net) -> RedC41
- U206 pad 2: (no net) -> RedC43
- U206 pad 3: (no net) -> RedC44
- U206 pad 4: (no net) -> RedC45
- U206 pad 5: (no net) -> RedC46
- U206 pad 6: (no net) -> RedC47
- U206 pad 7: (no net) -> RedC48
- U206 pad 9: N-0000024 -> N-00000199
- U207 pad 1: (no net) -> RedC50
- U207 pad 10: VCC -> N-00000273
- U207 pad 13: GND -> N-00000302
- U207 pad 14: N-0000024 -> N-00000258
- U207 pad 15: (no net) -> RedC49
- U207 pad 2: (no net) -> RedC51
- U207 pad 3: (no net) -> RedC52
- U207 pad 4: (no net) -> RedC53
- U207 pad 5: (no net) -> RedC54
- U207 pad 6: (no net) -> RedC55
- U207 pad 7: (no net) -> RedC56
- U207 pad 9: N-0000014 -> N-00000200
- U208 pad 1: (no net) -> RedC58
- U208 pad 10: VCC -> N-00000276
- U208 pad 13: GND -> N-00000275
- U208 pad 14: N-0000014 -> N-00000257
- U208 pad 15: (no net) -> RedC57
- U208 pad 2: (no net) -> RedC59
- U208 pad 3: (no net) -> RedC60
- U208 pad 4: (no net) -> RedC61
- U208 pad 5: (no net) -> RedC62
- U208 pad 6: (no net) -> RedC63
- U208 pad 7: (no net) -> RedC64
- U208 pad 9: (no net) -> /ColorControl/NextColor
Routing:
- net VCC: track 0.00 -> 268.4 mm, vias 0 -> 17
- net SRCLK: track 0.00 -> 244.3 mm
- net LATCH: track 0.00 -> 219.5 mm, vias 0 -> 9
- net AnodePlane1: track 0.00 -> 128.0 mm, vias 0 -> 1
- net /AnodeControl/AnodeP8: track 0.00 -> 115.2 mm, vias 0 -> 1
- net GND: track 0.00 -> 108.8 mm, vias 0 -> 9
- net /AnodeControl/AnodeP7: track 0.00 -> 103.1 mm, vias 0 -> 1
- net AnodePlane2: track 0.00 -> 98.8 mm, vias 0 -> 1
- net /AnodeControl/AnodeP6: track 0.00 -> 92.2 mm, vias 0 -> 1
- net AnodePlane3: track 0.00 -> 85.2 mm, vias 0 -> 1
- net /AnodeControl/AnodeP5: track 0.00 -> 80.8 mm, vias 0 -> 1
- net AnodePlane4: track 0.00 -> 72.4 mm, vias 0 -> 1
- net /AnodeControl/AnodeP4: track 0.00 -> 69.5 mm, vias 0 -> 1
- net AnodePlane5: track 0.00 -> 59.6 mm, vias 0 -> 1
- net /AnodeControl/AnodeP3: track 0.00 -> 57.7 mm, vias 0 -> 1
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- added copper zone on B.Cu, net GND
- added copper zone on F.Cu, net VCC
Other:
- board outline added: 169.6 x 61.6 mm
