File: 8x8x8LEDCube/8x8x8LEDCube.sch (KiCad schematic (older format))
At the start: 1 part, among them P101 CONN_2

Commit message: Final version of the PCB
Parts:
- added C101: CONNECTOR_1X64, symbol CONNECTOR_1X64
- added K101: CONN_3, symbol CONN_3
- added P102: CONN_2, symbol CONN_2
- added P103: CONN_8, symbol CONN_8
- added R101: 0, ~, symbol R
Connections:
- net RedControl/VCC renamed VCC
- new net: P102.1 (P1), P102.2 (PM), R101.1
- new net AnodeControl/AnodeP1: P103.1 (P1)
- new net AnodeControl/AnodeP2: P103.2 (P2)
- new net AnodeControl/AnodeP3: P103.3 (P3)
- new net AnodeControl/AnodeP4: P103.4 (P4)
- new net AnodeControl/AnodeP5: P103.5 (P5)
- new net AnodeControl/AnodeP6: P103.6 (P6)
- new net AnodeControl/AnodeP7: P103.7 (P7)
- new net AnodeControl/AnodeP8: P103.8 (P8)
- new net ColorControl/C10Red: C101.10
- new net ColorControl/C11Red: C101.11
- new net ColorControl/C12Red: C101.12
- new net ColorControl/C13Red: C101.13
- new net ColorControl/C14Red: C101.14
- new net ColorControl/C15Red: C101.15
- new net ColorControl/C16Red: C101.16
- new net ColorControl/C17Red: C101.17
- new net ColorControl/C18Red: C101.18
- new net ColorControl/C19Red: C101.19
- new net ColorControl/C1Red: C101.1
- new net ColorControl/C20Red: C101.20
- new net ColorControl/C21Red: C101.21
- new net ColorControl/C22Red: C101.22
- new net ColorControl/C23Red: C101.23
- new net ColorControl/C24Red: C101.24
- new net ColorControl/C25Red: C101.25
- new net ColorControl/C26Red: C101.26
- new net ColorControl/C27Red: C101.27
- new net ColorControl/C28Red: C101.28
- new net ColorControl/C29Red: C101.29
- new net ColorControl/C2Red: C101.2
- new net ColorControl/C30Red: C101.30
- new net ColorControl/C31Red: C101.31
- new net ColorControl/C32Red: C101.32
- new net ColorControl/C33Red: C101.33
- new net ColorControl/C34Red: C101.34
- new net ColorControl/C35Red: C101.35
- new net ColorControl/C36Red: C101.36
- new net ColorControl/C37Red: C101.37
- new net ColorControl/C38Red: C101.38
- new net ColorControl/C39Red: C101.39
- new net ColorControl/C3Red: C101.3
- new net ColorControl/C40Red: C101.40
- new net ColorControl/C41Red: C101.41
- new net ColorControl/C42Red: C101.42
- new net ColorControl/C43Red: C101.43
- new net ColorControl/C44Red: C101.44
- new net ColorControl/C45Red: C101.45
- new net ColorControl/C46Red: C101.46
- new net ColorControl/C47Red: C101.47
- new net ColorControl/C48Red: C101.48
- new net ColorControl/C49Red: C101.49
- new net ColorControl/C4Red: C101.4
- new net ColorControl/C50Red: C101.50
- new net ColorControl/C51Red: C101.51
- new net ColorControl/C52Red: C101.52
- new net ColorControl/C53Red: C101.53
- new net ColorControl/C54Red: C101.54
- new net ColorControl/C55Red: C101.55
- new net ColorControl/C56Red: C101.56
- new net ColorControl/C57Red: C101.57
- new net ColorControl/C58Red: C101.58
- new net ColorControl/C59Red: C101.59
- new net ColorControl/C5Red: C101.5
- new net ColorControl/C60Red: C101.60
- new net ColorControl/C61Red: C101.61
- new net ColorControl/C62Red: C101.62
- new net ColorControl/C63Red: C101.63
- new net ColorControl/C64Red: C101.64
- new net ColorControl/C6Red: C101.6
- new net ColorControl/C7Red: C101.7
- new net ColorControl/C8Red: C101.8
- new net ColorControl/C9Red: C101.9
- new net ColorControl/NextColor: R101.2
- new net DATA_IN: K101.1 (P1)
- new net LATCH: K101.2 (PM)
- new net SRCLK: K101.3 (P3)
Other:
- moved on the sheet: P101
