File: 8x8x8LEDCube/RedControl.sch (KiCad schematic (older format))
At the start: 40 parts, among them Q201 NPN, Q202 NPN, Q203 NPN, Q204 NPN, Q205 NPN, Q206 NPN, Q207 NPN, Q208 NPN, U201 SN74HC595DWR, U202 SN74HC595DWR, U203 SN74HC595DWR, U204 SN74HC595DWR, U205 SN74HC595DWR, U206 SN74HC595DWR, U207 SN74HC595DWR, U208 SN74HC595DWR

Commit message: Final version of the PCB
Parts:
- added C201, C202, C203, C204, C205, C206, C207, C208: 0.1u, ~, symbol C
- added Q209, Q210, Q211, Q212, Q213, Q214, Q215, Q216, Q217, Q218, Q219, Q220, Q221, Q222, Q223, Q224, Q225, Q226, Q227, Q228, Q229, Q230, Q231, Q232, Q233, Q234, Q235, Q236, Q237, Q238, Q239, Q240, Q241, Q242, Q243, Q244, Q245, Q246, Q247, Q248, Q249, Q250, Q251, Q252, Q253, Q254, Q255, Q256, Q257, Q258, Q259, Q260, Q261, Q262, Q263, Q264: NPN, ~, symbol NPN
- added R201, R202, R203, R204, R205, R206, R207, R208, R209, R210, R211, R212, R213, R214, R215, R216, R409, R410, R411, R412, R413, R414, R415, R416, R444: 0, ~, symbol R
- added R241, R242, R244, R245, R247, R248, R250, R251, R253, R254, R256, R257, R259, R260, R262, R263, R265, R266, R268, R269, R271, R272, R274, R275, R277, R278, R280, R281, R283, R284, R286, R287, R289, R290, R292, R293, R295, R296, R298, R299, R301, R302, R304, R305, R307, R308, R310, R311, R313, R314, R316, R317, R319, R320, R322, R323, R325, R326, R328, R329, R331, R332, R334, R335, R337, R338, R340, R341, R343, R344, R346, R347, R349, R350, R352, R353, R355, R356, R358, R359, R361, R362, R364, R365, R367, R368, R370, R371, R373, R374, R376, R377, R379, R380, R382, R383, R385, R386, R388, R389, R391, R392, R394, R395, R397, R398, R400, R401, R403, R404, R406, R407: 1K, ~, symbol R
- added R243, R246, R249, R252, R255, R258, R261, R264, R267, R270, R273, R276, R279, R282, R285, R288, R291, R294, R297, R300, R303, R306, R309, R312, R315, R318, R321, R324, R327, R330, R333, R336, R339, R342, R345, R348, R351, R354, R357, R360, R363, R366, R369, R372, R375, R378, R381, R384, R387, R390, R393, R396, R399, R402, R405, R408: 100, ~, symbol R
- renumbered R201 to R217, R202 to R218, R203 to R219, R204 to R220, R205 to R221, R206 to R222, R207 to R223, R208 to R224, R209 to R225, R210 to R226, R211 to R227, R212 to R228, R213 to R229, R214 to R230, R215 to R231, R216 to R232, R217 to R233, R218 to R234, R219 to R235, R220 to R236, R221 to R237, R222 to R238, R223 to R239, R224 to R240
Connections:
- net DATA_IN: now also R416.1; no longer U201.14 (SER)
- net GND: now also C201.2, C202.2, C203.2, C204.2, C205.2, C206.2, C207.2, C208.2, Q209.1 (E), Q210.1 (E), Q211.1 (E), Q212.1 (E), Q213.1 (E), Q214.1 (E), Q215.1 (E), Q216.1 (E), Q217.1 (E), Q218.1 (E), Q219.1 (E), Q220.1 (E), Q221.1 (E), Q222.1 (E), Q223.1 (E), Q224.1 (E), Q225.1 (E), Q226.1 (E), Q227.1 (E), Q228.1 (E), Q229.1 (E), Q230.1 (E), Q231.1 (E), Q232.1 (E), Q233.1 (E), Q234.1 (E), Q235.1 (E), Q236.1 (E), Q237.1 (E), Q238.1 (E), Q239.1 (E), Q240.1 (E), Q241.1 (E), Q242.1 (E), Q243.1 (E), Q244.1 (E), Q245.1 (E), Q246.1 (E), Q247.1 (E), Q248.1 (E), Q249.1 (E), Q250.1 (E), Q251.1 (E), Q252.1 (E), Q253.1 (E), Q254.1 (E), Q255.1 (E), Q256.1 (E), Q257.1 (E), Q258.1 (E), Q259.1 (E), Q260.1 (E), Q261.1 (E), Q262.1 (E), Q263.1 (E), Q264.1 (E), R202.1, R204.1, R206.1, R208.1, R210.1, R212.1, R214.1, R216.1; no longer U201.13 (~OE), U202.13 (~OE), U203.13 (~OE), U205.13 (~OE), U206.13 (~OE), U207.13 (~OE), U208.13 (~OE)
- net VCC: now also C201.1, C202.1, C203.1, C204.1, C205.1, C206.1, C207.1, C208.1, R201.1, R203.1, R205.1, R207.1, R209.1, R211.1, R213.1, R215.1, R242.1, R245.1, R248.1, R251.1, R254.1, R257.1, R260.1, R263.1, R266.1, R269.1, R272.1, R275.1, R278.1, R281.1, R284.1, R287.1, R290.1, R293.1, R296.1, R299.1, R302.1, R305.1, R308.1, R311.1, R314.1, R317.1, R320.1, R323.1, R326.1, R329.1, R332.1, R335.1, R338.1, R341.1, R344.1, R347.1, R350.1, R353.1, R356.1, R359.1, R362.1, R365.1, R368.1, R371.1, R374.1, R377.1, R380.1, R383.1, R386.1, R389.1, R392.1, R395.1, R398.1, R401.1, R404.1, R407.1; no longer U201.10 (~SRCLR), U202.10 (~SRCLR), U203.10 (~SRCLR), U204.10 (~SRCLR), U205.10 (~SRCLR), U206.10 (~SRCLR), U207.10 (~SRCLR), U208.10 (~SRCLR)
- net at U201.9 (QH'): now also R415.2; no longer U202.14 (SER)
- net RedC10: now reaches U202.1 (QB)
- net RedC10: now also R244.1
- net RedC9: now reaches U202.15 (QA)
- net RedC9: now also R241.1
- net RedC11: now reaches U202.2 (QC)
- net RedC11: now also R247.1
- net RedC12: now reaches U202.3 (QD)
- net RedC12: now also R250.1
- net RedC13: now reaches U202.4 (QE)
- net RedC13: now also R253.1
- net RedC14: now reaches U202.5 (QF)
- net RedC14: now also R256.1
- net RedC15: now reaches U202.6 (QG)
- net RedC15: now also R259.1
- net RedC16: now reaches U202.7 (QH)
- net RedC16: now also R262.1
- net at U202.9 (QH'): now also R412.2; no longer U203.14 (SER)
- net RedC18: now reaches U203.1 (QB)
- net RedC18: now also R268.1
- net RedC17: now reaches U203.15 (QA)
- net RedC17: now also R265.1
- net RedC19: now reaches U203.2 (QC)
- net RedC19: now also R271.1
- net RedC20: now reaches U203.3 (QD)
- net RedC20: now also R274.1
- net RedC21: now reaches U203.4 (QE)
- net RedC21: now also R277.1
- net RedC22: now reaches U203.5 (QF)
- net RedC22: now also R280.1
- net RedC23: now reaches U203.6 (QG)
- net RedC23: now also R283.1
- net RedC24: now reaches U203.7 (QH)
- net RedC24: now also R286.1
- net at U203.9 (QH'): now also R413.2; no longer U204.14 (SER)
- net RedC26: now reaches U204.1 (QB)
- net RedC26: now also R292.1
- net at U204.13 (~OE): now also R208.2
- net RedC25: now reaches U204.15 (QA)
- net RedC25: now also R289.1
- net RedC27: now reaches U204.2 (QC)
- net RedC27: now also R295.1
- net RedC28: now reaches U204.3 (QD)
- net RedC28: now also R298.1
- net RedC29: now reaches U204.4 (QE)
- net RedC29: now also R301.1
- net RedC30: now reaches U204.5 (QF)
- net RedC30: now also R304.1
- net RedC31: now reaches U204.6 (QG)
- net RedC31: now also R307.1
- net RedC32: now reaches U204.7 (QH)
- net RedC32: now also R310.1
- net at U204.9 (QH'): now also R414.2; no longer U205.14 (SER)
- net RedC34: now reaches U205.1 (QB)
- net RedC34: now also R316.1
- net RedC33: now reaches U205.15 (QA)
- net RedC33: now also R313.1
- net RedC35: now reaches U205.2 (QC)
- net RedC35: now also R319.1
- net RedC36: now reaches U205.3 (QD)
- net RedC36: now also R322.1
- net RedC37: now reaches U205.4 (QE)
- net RedC37: now also R325.1
- net RedC38: now reaches U205.5 (QF)
- net RedC38: now also R328.1
- net RedC39: now reaches U205.6 (QG)
- net RedC39: now also R331.1
- net RedC40: now reaches U205.7 (QH)
- net RedC40: now also R334.1
- net at U205.9 (QH'): now also R409.2; no longer U206.14 (SER)
- net RedC42: now reaches U206.1 (QB)
- net RedC42: now also R340.1
- net RedC41: now reaches U206.15 (QA)
- net RedC41: now also R337.1
- net RedC43: now reaches U206.2 (QC)
- net RedC43: now also R343.1
- net RedC44: now reaches U206.3 (QD)
- net RedC44: now also R346.1
- net RedC45: now reaches U206.4 (QE)
- net RedC45: now also R349.1
- net RedC46: now reaches U206.5 (QF)
- net RedC46: now also R352.1
- net RedC47: now reaches U206.6 (QG)
- net RedC47: now also R355.1
- net RedC48: now reaches U206.7 (QH)
- net RedC48: now also R358.1
- net at U206.9 (QH'): now also R410.2; no longer U207.14 (SER)
- net RedC50: now reaches U207.1 (QB)
- net RedC50: now also R364.1
- net RedC49: now reaches U207.15 (QA)
- net RedC49: now also R361.1
- net RedC51: now reaches U207.2 (QC)
- net RedC51: now also R367.1
- net RedC52: now reaches U207.3 (QD)
- net RedC52: now also R370.1
- net RedC53: now reaches U207.4 (QE)
- net RedC53: now also R373.1
- net RedC54: now reaches U207.5 (QF)
- net RedC54: now also R376.1
- net RedC55: now reaches U207.6 (QG)
- net RedC55: now also R379.1
- net RedC56: now reaches U207.7 (QH)
- net RedC56: now also R382.1
- net at U207.9 (QH'): now also R411.2; no longer U208.14 (SER)
- net RedC58: now reaches U208.1 (QB)
- net RedC58: now also R388.1
- net RedC57: now reaches U208.15 (QA)
- net RedC57: now also R385.1
- net RedC59: now reaches U208.2 (QC)
- net RedC59: now also R391.1
- net RedC60: now reaches U208.3 (QD)
- net RedC60: now also R394.1
- net RedC61: now reaches U208.4 (QE)
- net RedC61: now also R397.1
- net RedC62: now reaches U208.5 (QF)
- net RedC62: now also R400.1
- net RedC63: now reaches U208.6 (QG)
- net RedC63: now also R403.1
- net RedC64: now reaches U208.7 (QH)
- net RedC64: now also R406.1
- net NextColor: now reaches U208.9 (QH')
- new net: R201.2, U201.10 (~SRCLR)
- new net: R202.2, U201.13 (~OE)
- new net: R416.2, R444.2, U201.14 (SER)
- new net: R203.2, U202.10 (~SRCLR)
- new net: R204.2, U202.13 (~OE)
- new net: R415.1, U202.14 (SER)
- new net: R205.2, U203.10 (~SRCLR)
- new net: R206.2, U203.13 (~OE)
- new net: R412.1, U203.14 (SER)
- new net: R207.2, U204.10 (~SRCLR)
- new net: R413.1, U204.14 (SER)
- new net: R209.2, U205.10 (~SRCLR)
- new net: R210.2, U205.13 (~OE)
- new net: R414.1, U205.14 (SER)
- new net: R211.2, U206.10 (~SRCLR)
- new net: R212.2, U206.13 (~OE)
- new net: R409.1, U206.14 (SER)
- new net: R213.2, U207.10 (~SRCLR)
- new net: R214.2, U207.13 (~OE)
- new net: R410.1, U207.14 (SER)
- new net: R215.2, U208.10 (~SRCLR)
- new net: R216.2, U208.13 (~OE)
- new net: R411.1, U208.14 (SER)
- new net: Q209.2 (B), R241.2
- new net: Q209.3 (C), R242.2, R243.1
- new net: Q210.2 (B), R244.2
- new net: Q210.3 (C), R245.2, R246.1
- new net: Q211.2 (B), R247.2
- new net: Q211.3 (C), R248.2, R249.1
- new net: Q212.2 (B), R250.2
- new net: Q212.3 (C), R251.2, R252.1
- new net: Q213.2 (B), R253.2
- new net: Q213.3 (C), R254.2, R255.1
- new net: Q214.2 (B), R256.2
- new net: Q214.3 (C), R257.2, R258.1
- new net: Q215.2 (B), R259.2
- new net: Q215.3 (C), R260.2, R261.1
- new net: Q216.2 (B), R262.2
- new net: Q216.3 (C), R263.2, R264.1
- new net: Q225.2 (B), R289.2
- new net: Q225.3 (C), R290.2, R291.1
- new net: Q226.2 (B), R292.2
- new net: Q226.3 (C), R293.2, R294.1
- new net: Q227.2 (B), R295.2
- new net: Q227.3 (C), R296.2, R297.1
- new net: Q228.2 (B), R298.2
- new net: Q228.3 (C), R299.2, R300.1
- new net: Q229.2 (B), R301.2
- new net: Q229.3 (C), R302.2, R303.1
- new net: Q230.2 (B), R304.2
- new net: Q230.3 (C), R305.2, R306.1
- new net: Q231.2 (B), R307.2
- new net: Q231.3 (C), R308.2, R309.1
- new net: Q232.2 (B), R310.2
- new net: Q232.3 (C), R311.2, R312.1
- new net: Q217.2 (B), R265.2
- new net: Q217.3 (C), R266.2, R267.1
- new net: Q218.2 (B), R268.2
- new net: Q218.3 (C), R269.2, R270.1
- new net: Q219.2 (B), R271.2
- new net: Q219.3 (C), R272.2, R273.1
- new net: Q220.2 (B), R274.2
- new net: Q220.3 (C), R275.2, R276.1
- new net: Q221.2 (B), R277.2
- new net: Q221.3 (C), R278.2, R279.1
- new net: Q222.2 (B), R280.2
- new net: Q222.3 (C), R281.2, R282.1
- new net: Q223.2 (B), R283.2
- new net: Q223.3 (C), R284.2, R285.1
- new net: Q224.2 (B), R286.2
- new net: Q224.3 (C), R287.2, R288.1
- new net: Q233.2 (B), R313.2
- new net: Q233.3 (C), R314.2, R315.1
- new net: Q234.2 (B), R316.2
- new net: Q234.3 (C), R317.2, R318.1
- new net: Q235.2 (B), R319.2
- new net: Q235.3 (C), R320.2, R321.1
- new net: Q236.2 (B), R322.2
- new net: Q236.3 (C), R323.2, R324.1
- new net: Q237.2 (B), R325.2
- new net: Q237.3 (C), R326.2, R327.1
- new net: Q238.2 (B), R328.2
- new net: Q238.3 (C), R329.2, R330.1
- new net: Q239.2 (B), R331.2
- new net: Q239.3 (C), R332.2, R333.1
- new net: Q240.2 (B), R334.2
- new net: Q240.3 (C), R335.2, R336.1
- new net: Q241.2 (B), R337.2
- new net: Q241.3 (C), R338.2, R339.1
- new net: Q242.2 (B), R340.2
- new net: Q242.3 (C), R341.2, R342.1
- new net: Q243.2 (B), R343.2
- new net: Q243.3 (C), R344.2, R345.1
- new net: Q244.2 (B), R346.2
- new net: Q244.3 (C), R347.2, R348.1
- new net: Q245.2 (B), R349.2
- new net: Q245.3 (C), R350.2, R351.1
- new net: Q246.2 (B), R352.2
- new net: Q246.3 (C), R353.2, R354.1
- new net: Q247.2 (B), R355.2
- new net: Q247.3 (C), R356.2, R357.1
- new net: Q248.2 (B), R358.2
- new net: Q248.3 (C), R359.2, R360.1
- new net: Q249.2 (B), R361.2
- new net: Q249.3 (C), R362.2, R363.1
- new net: Q250.2 (B), R364.2
- new net: Q250.3 (C), R365.2, R366.1
- new net: Q251.2 (B), R367.2
- new net: Q251.3 (C), R368.2, R369.1
- new net: Q252.2 (B), R370.2
- new net: Q252.3 (C), R371.2, R372.1
- new net: Q253.2 (B), R373.2
- new net: Q253.3 (C), R374.2, R375.1
- new net: Q254.2 (B), R376.2
- new net: Q254.3 (C), R377.2, R378.1
- new net: Q255.2 (B), R379.2
- new net: Q255.3 (C), R380.2, R381.1
- new net: Q256.2 (B), R382.2
- new net: Q256.3 (C), R383.2, R384.1
- new net: Q257.2 (B), R385.2
- new net: Q257.3 (C), R386.2, R387.1
- new net: Q258.2 (B), R388.2
- new net: Q258.3 (C), R389.2, R390.1
- new net: Q259.2 (B), R391.2
- new net: Q259.3 (C), R392.2, R393.1
- new net: Q260.2 (B), R394.2
- new net: Q260.3 (C), R395.2, R396.1
- new net: Q261.2 (B), R397.2
- new net: Q261.3 (C), R398.2, R399.1
- new net: Q262.2 (B), R400.2
- new net: Q262.3 (C), R401.2, R402.1
- new net: Q263.2 (B), R403.2
- new net: Q263.3 (C), R404.2, R405.1
- new net: Q264.2 (B), R406.2
- new net: Q264.3 (C), R407.2, R408.1
- new net C10Red: R246.2
- new net C11Red: R249.2
- new net C12Red: R252.2
- new net C13Red: R255.2
- new net C14Red: R258.2
- new net C15Red: R261.2
- new net C16Red: R264.2
- new net C17Red: R267.2
- new net C18Red: R270.2
- new net C19Red: R273.2
- new net C20Red: R276.2
- new net C21Red: R279.2
- new net C22Red: R282.2
- new net C23Red: R285.2
- new net C24Red: R288.2
- new net C25Red: R291.2
- new net C26Red: R294.2
- new net C27Red: R297.2
- new net C28Red: R300.2
- new net C29Red: R303.2
- new net C30Red: R306.2
- new net C31Red: R309.2
- new net C32Red: R312.2
- new net C33Red: R315.2
- new net C34Red: R318.2
- new net C35Red: R321.2
- new net C36Red: R324.2
- new net C37Red: R327.2
- new net C38Red: R330.2
- new net C39Red: R333.2
- new net C40Red: R336.2
- new net C41Red: R339.2
- new net C42Red: R342.2
- new net C43Red: R345.2
- new net C44Red: R348.2
- new net C45Red: R351.2
- new net C46Red: R354.2
- new net C47Red: R357.2
- new net C48Red: R360.2
- new net C49Red: R363.2
- new net C50Red: R366.2
- new net C51Red: R369.2
- new net C52Red: R372.2
- new net C53Red: R375.2
- new net C54Red: R378.2
- new net C55Red: R381.2
- new net C56Red: R384.2
- new net C57Red: R387.2
- new net C58Red: R390.2
- new net C59Red: R393.2
- new net C60Red: R396.2
- new net C61Red: R399.2
- new net C62Red: R402.2
- new net C63Red: R405.2
- new net C64Red: R408.2
- new net C9Red: R243.2
- new net FIRST_COLOR: R444.1
Other:
- note added: "Esta resistencia se pondrá solo cuando sea el primer color a controlar.\nEs decir, solo cuando va después del control de los ánodos comunes."
- note added: "PARA EL CANAL ROJO LAS RESISTENCIAS CONECTADAS AL COLECTOR DE LOS\nTRANSISTORES ES DE 100 ohm, PERO PARA LOS CANALES VERDE Y AZUL LA \nrESISTENCIA TIENE QUE SER DE 50ohm. HAY QUE TENER EN CUENTA ESO PARA\nEL PEDIDO, PUESTO QUE EL ESQUEMÁTICO ES EL MISMO"
- note added: "R416 se pondrá solo cuando la placa controle solo un color.\nEs decir, cuando no se utilice la parte de control de los ánodos.\nEn este caso la señal vendrá de la clema, del polo DATA_IN"
